Commit message: Fixed inertial parameters, added basic simulation systems

File: src/ostem_bringup/urdf/ostem.urdf.xacro (robot description, xacro)
@@ -3,4 +3,6 @@
     <!-- Main robot structure -->
     <xacro:include filename="ostem_core.xacro" />
+    <!-- Robot kinematics -->
+    <xacro:include filename="ostem_gazebo_kinematics.xacro" />
     <!-- Sensors -->
     <gazebo>

File: src/ostem_bringup/urdf/ostem_core.xacro (robot description, xacro)
@@ -71,10 +71,10 @@
         </collision>
         <inertial>
-            <mass value="${wheel_mass}" />
-            <origin xyz="0 0 0" rpy="${pi/2} 0 0" />
+            <origin xyz="${0.225-(chassis_length/2)} ${0.207-(chassis_breadth/2)} ${0.129-(chassis_height/2)}" rpy="0 0 0" />
+            <mass value="${chassis_mass}" />
             <inertia
-                ixx="${1/12*wheel_mass*(3*(wheel_radius*wheel_radius)+(wheel_length*wheel_length))}"
-                iyy="${1/12*wheel_mass*(3*(wheel_radius*wheel_radius)+(wheel_length*wheel_length))}"
-                izz="${1/2*wheel_mass*(wheel_radius*wheel_radius)}"
+                ixx="0.143"
+                iyy="0.176"
+                izz="0.230"
                 ixy="0.0" iyz="0.0" ixz="0.0" />
         </inertial>
